File: KICAD/DS2_Addon.sch (KiCad schematic (older format))
At the start: 31 parts, among them J1 MCU, J2 Analog1, J3 Conn_01x03, J4 Reference, J5 Analog2, U1 ADS122U04

Commit message: working version for getting basic data for the thesis
Parts:
- JP1, JP2, JP3, JP4: symbol Device:Jumper_NO_Small -> DS2_Addon-rescue:Jumper_NO_Small-Device
Connections:
- net ~RESET renamed ~{RESET}
